File: pinbot-carrier.kicad_sch (KiCad schematic)
At the start: 118 parts, among them J1 USB4105-GF-A-120, J2 Conn_02x20_Odd_Even, J3 HC-1.0-4PWT, J4 SM06B-SRSS-TB, J5 USB_A, J6 USB_A, J7 USB_A, K1 EC2-5SNU, K2 EC2-5SNU, K3 EC2-5SNU, K4 EC2-5SNU, U1 TCA9535PWR, U10 ZXBM5210-S, U11 ZXBM5210-S, U12 ZXBM5210-S, U13 MIC2026-2xM, U14 USBLC6-2SC6, U15 USBLC6-2SC6, U16 USBLC6-2SC6, U17 USBLC6-2SC6, U18 FE1.1s, U19 MIC2026-2xM, U2 ADS1015IDGS, U7 ADS1015IDGS, U8 74HC04, U9 ZXBM5210-S, Y1 12MHz

Commit message: r0.2 remade from a scratch
Parts:
- removed C10, C20, C21, C22, C23, C5, C7, C9: 0.1uFx50V, Capacitor_SMD:C_0603_1608Metric, symbol Device:C_Small
- removed C11, C15, C16: 10uFx10V, Capacitor_SMD:C_0603_1608Metric, symbol Device:C_Small
- removed C13, C14, C3, C8: 100uFx16V, Capacitor_SMD:CP_Elec_6.3x5.4, symbol Device:C_Polarized_Small
- removed D1, D2, D3, D7, D8, D9: LTST-S270KGKT, LED_0603_1608Metric_side:LED_0603_1608Metric_side, symbol Device:LED
- removed D10, D11, D12, D13, D14, D15, D16, D17: ESD5Z3.3T5G, Diode_SMD:D_SOD-523, symbol Diode:ESD5Zxx
- removed J3: HC-1.0-4PWT, Connector_JST:JST_SH_SM04B-SRSS-TB_1x04-1MP_P1.00mm_Horizontal, symbol Connector_Generic:Conn_01x04
- removed J4: SM06B-SRSS-TB, SM06B-SRSS-TB:JST_SM06B-SRSS-TB, symbol Connector_Generic:Conn_01x06
- removed JP1, JP2: SolderJumper_2_Open, Jumper:SolderJumper-2_P1.3mm_Open_RoundedPad1.0x1.5mm, symbol Jumper:SolderJumper_2_Open
- removed K1, K2, K3, K4: EC2-5SNU, Relay_THT:Relay_DPDT_Kemet_EC2, symbol Relay:EC2-5SNU
- removed R1, R12, R13, R2, R3: 820k, Resistor_SMD:R_0603_1608Metric, symbol Device:R_Small
- removed R16, R17, R20, R25, R6, R8, R9: 120k, Resistor_SMD:R_0603_1608Metric, symbol Device:R_Small
- removed R21, R24, R26, R27, R35, R36, R37: 10k, Resistor_SMD:R_0603_1608Metric, symbol Device:R_Small
- removed R29, R30, R31, R32, R39, R40, R41: 330R, Resistor_SMD:R_0603_1608Metric, symbol Device:R_Small
- removed R38: 2.7k, Resistor_SMD:R_0603_1608Metric, symbol Device:R_Small
- removed U10, U11, U12, U9: ZXBM5210-S, Package_SO:SOIC-8_3.9x4.9mm_P1.27mm, symbol Driver_Motor:ZXBM5210-S
- removed U13, U19: MIC2026-2xM, Package_SO:SOIC-8_3.9x4.9mm_P1.27mm, symbol Power_Management:MIC2026-2xM
- removed U18: FE1.1s, Package_SO:SSOP-28_3.9x9.9mm_P0.635mm, symbol Interface_USB:FE1.1s
- removed U2, U7: ADS1015IDGS, Package_SO:TSSOP-10_3x3mm_P0.5mm, symbol Analog_ADC:ADS1015IDGS
- removed U8: 74HC04, Package_SO:SOIC-14_3.9x8.7mm_P1.27mm, symbol 74xx:74HC04
- removed Y1: 12MHz, Crystal:Crystal_SMD_3225-4Pin_3.2x2.5mm, symbol Device:Crystal_GND24
- added C10, C36, C37: 100uFx10V, Capacitor_Tantalum_SMD:CP_EIA-3528-21_Kemet-B, symbol Device:C_Polarized_Small
- added C2, C8: 0.1uFx50V, Capacitor_SMD:C_0603_1608Metric, symbol Device:C_Small
- added C25: 10uFx10V, Capacitor_SMD:C_0603_1608Metric, symbol Device:C_Small
- added D1, D19, D2, D20, D21, D22, D23, D24: ESD5Z3.3T5G, Diode_SMD:D_SOD-523, symbol Diode:ESD5Zxx
- added D15: LTST-S270KRKT, LED_0603_1608Metric_side:LED_0603_1608Metric_side, symbol Device:LED
- added D16: LTST-S270KGKT, LED_0603_1608Metric_side:LED_0603_1608Metric_side, symbol Device:LED
- added D17: 19-21/GHC-YR1S2/4T, LED_SMD:LED_0603_1608Metric, symbol Device:LED
- added D48: SMAJ5.0A, Diode_SMD:D_SMA, symbol Diode:SMAJ5.0A
- added D49, D50: XL-1608SURC-06, LED_SMD:LED_0603_1608Metric, symbol Device:LED
- added D52, D53, D54, D55: BAT54S, Package_TO_SOT_SMD:SOT-23, symbol Diode:BAT54S
- added F2, F3, F4, F5, F6, F8: MF-NSMF110-2, Fuse:Fuse_1206_3216Metric, symbol Device:Fuse
- added FID1, FID2: Fiducial, Fiducial:Fiducial_1mm_Mask2mm, symbol Mechanical:Fiducial
- added J3: Raspberry_Pi_4, Connector_PinHeader_2.54mm:PinHeader_2x20_P2.54mm_Vertical, symbol Connector:Raspberry_Pi_4
- added J4: Conn_02x20_Odd_Even, Connector_PinHeader_2.54mm:PinHeader_2x20_P2.54mm_Vertical, symbol Connector_Generic:Conn_02x20_Odd_Even
- added J5: SM06B-SRSS-TB, SM06B-SRSS-TB:JST_SM06B-SRSS-TB, symbol Connector_Generic:Conn_01x06
- added J6: HC-1.0-4PWT, Connector_JST:JST_SH_SM04B-SRSS-TB_1x04-1MP_P1.00mm_Horizontal, symbol Connector_Generic:Conn_01x04
- added R64, R65, R77, R78: 330R, Resistor_SMD:R_0603_1608Metric, symbol Device:R_Small
- added R80: 0, Resistor_SMD:R_0603_1608Metric, symbol Device:R_Small
- added TP10: 3V3, JLCImport:TestPoint_Loop_D1.80mm_Drill1.0mm_Beaded, symbol Connector:TestPoint
- added TP11: RPI_D+, JLCImport:TestPoint_Loop_D1.80mm_Drill1.0mm_Beaded, symbol Connector:TestPoint
- added TP12: RPI_D-, JLCImport:TestPoint_Loop_D1.80mm_Drill1.0mm_Beaded, symbol Connector:TestPoint
- added TP2: +5V, JLCImport:TestPoint_Loop_D1.80mm_Drill1.0mm_Beaded, symbol Connector:TestPoint
- added TP3: D-, JLCImport:TestPoint_Loop_D1.80mm_Drill1.0mm_Beaded, symbol Connector:TestPoint
- added TP4: D+, JLCImport:TestPoint_Loop_D1.80mm_Drill1.0mm_Beaded, symbol Connector:TestPoint
- added TP5: GND, JLCImport:TestPoint_Loop_D1.80mm_Drill1.0mm_Beaded, symbol Connector:TestPoint
- added TP6: SDA, JLCImport:TestPoint_Loop_D1.80mm_Drill1.0mm_Beaded, symbol Connector:TestPoint
- added TP7: SCL, JLCImport:TestPoint_Loop_D1.80mm_Drill1.0mm_Beaded, symbol Connector:TestPoint
- added U12: USBLC6-2SC6, Package_TO_SOT_SMD:SOT-23-6, symbol Power_Protection:USBLC6-2SC6
- added U3: TCA9535PWR, Package_SO:TSSOP-24_4.4x7.8mm_P0.65mm, symbol Interface_Expansion:TCA9535PWR
- A1: Check_prices (none) -> C33545975; LCSC Part # (none) -> C2977589; now left out of the parts list
- C1: renamed from C2; now not fitted
- C6: value 0.1uFx50V -> 10uFx10V; LCSC Part # C282519 -> C2959727; Mouser Part # CGA3E2X7R1H104M080AA -> GRM188Z71A106MA73J
- C9: renamed from C12; value 100uFx16V -> 100uFx10V; footprint Capacitor_SMD:CP_Elec_6.3x5.4 -> Capacitor_Tantalum_SMD:CP_EIA-3528-21_Kemet-B; LCSC Part # C129250 -> C600583; Mouser Part # UWT1C101MCL1GB -> (none)
- D4, D6: value LTST-S270KGKT -> 19-21/GHC-YR1S2/4T; footprint LED_0603_1608Metric_side:LED_0603_1608Metric_side -> LED_SMD:LED_0603_1608Metric; LCSC Part # C125113 -> C2986048; Mouser Part # LTST-S270KGKT -> (none)
- D5: value LTST-S270KRKT -> 19-21/GHC-YR1S2/4T; footprint LED_0603_1608Metric_side:LED_0603_1608Metric_side -> LED_SMD:LED_0603_1608Metric; LCSC Part # C125114 -> C2986048; Mouser Part # LTST-S270KRKT -> (none)
- H1, H2, H3, H4: footprint MountingHoles:MountingHole_3.2mm_M3_keepouts -> JLCImport:MountingHole_2.7mm; now fitted; now left out of the parts list
- J2: footprint Connector_PinSocket_2.54mm:PinSocket_2x20_P2.54mm_Vertical -> Connector_PinHeader_2.54mm:PinHeader_2x20_P2.54mm_Horizontal; LCSC Part # C2977589 -> C124369; now not fitted
- J7: renamed from J5; Manufacturer Part (none) -> USB1125-GF-B
- J8: renamed from J6; Manufacturer Part (none) -> USB1125-GF-B
- J9: renamed from J7; Manufacturer Part (none) -> USB1125-GF-B
- R1: renamed from R7; now not fitted
- R14, R15, R4: value 820k -> 330R; LCSC Part # C2907070 -> C23138; Mouser Part # ERJ-3EKF8203V -> RMCF0603FT330R
- R16: renamed from R42; LCSC Part # C2907113 -> C98220
- R17: renamed from R43; LCSC Part # C2907113 -> C98220
- R18, R19: LCSC Part # C2907113 -> C98220
- R22, R23: value 10k -> 0; LCSC Part # C2907113 -> C95177; Mouser Part # RMC1/16K1002DTP -> ERJ-3EKF5101V; now not fitted; now left out of the parts list
- R5: value 120k -> 330R; LCSC Part # C2930027 -> C23138; Mouser Part # CRGCQ0603F120K -> RMCF0603FT330R
- U1: renamed from U17; Manufacturer Part (none) -> USBLC6-2SC6-ES
- U2: renamed from U1; Manufacturer Part (none) -> TCA9535PWR(UMW)
- U4: renamed from U14; Manufacturer Part (none) -> USBLC6-2SC6-ES
- U5: renamed from U15; Manufacturer Part (none) -> USBLC6-2SC6-ES
- U6: renamed from U16; Manufacturer Part (none) -> USBLC6-2SC6-ES
- renumbered C17 to C12, C18 to C13, C19 to C14, C1 to C7, R10 to R2, R33 to R20, R34 to R21, R28 to R24, R11 to R3
Connections:
- net COM1 is gone; now on net GND: J2.9 (Pin_9)
- net COM2 is gone; now on net GPIO5_OUT: J2.15 (Pin_15)
- net NC1 is gone; now on net GPIO0_OUT: J2.12 (Pin_12)
- net NC2 is gone; now on net GPIO6_OUT: J2.18 (Pin_18)
- net NO1 is gone; now on net GND: J2.10 (Pin_10)
- net NO2 is gone; now on net GPIO4_OUT: J2.16 (Pin_16)
- net +3V3: now also R18.1, R19.1, C8.2, D52.2 (K), D53.2 (K), D54.2 (K), D55.2 (K), F4.2, F5.1, F8.2, R78.2, TP10.1, U3.21 (A0), U3.24 (VCC); no longer C6.2, J2.34 (Pin_34)
- net +5V: now also A1.2 (+5V), A1.4 (+5V), C6.2, R14.1, R15.1, R4.1, R5.1, C25.2, F2.2, F3.2, F6.1, R77.2, TP2.1, U12.5 (VBUS); no longer J2.29 (Pin_29)
- net +5V_USB2: now also C36.1
- net +5V_USB3: now also C37.1
- net +5V_USB4: now also J2.38 (Pin_38), C10.1, C2.2; no longer J2.33 (Pin_33)
- net 1D+: now also R22.2
- net 1D-: now also R23.2
- net 4O_D+: now also J2.40 (Pin_40); no longer J2.39 (Pin_39)
- net 4O_D-: now also J2.39 (Pin_39); no longer J2.40 (Pin_40)
- net AN0: now also J2.2 (Pin_2); no longer J2.1 (Pin_1)
- net AN1: now also J2.1 (Pin_1); no longer J2.2 (Pin_2)
- net AN2: now also J2.4 (Pin_4); no longer J2.3 (Pin_3)
- net AN3: now also J2.3 (Pin_3); no longer J2.4 (Pin_4), R4.1
- net AN4: now also J2.6 (Pin_6); no longer J2.5 (Pin_5)
- net AN5: now also J2.5 (Pin_5); no longer J2.6 (Pin_6)
- net AN6: now also J2.8 (Pin_8); no longer J2.7 (Pin_7), R14.1
- net AN7: now also J2.7 (Pin_7); no longer J2.8 (Pin_8), R15.1
- net GND: now also D5.1 (K), D6.1 (K), J2.19 (Pin_19), J2.20 (Pin_20), J2.35 (Pin_35), J2.36 (Pin_36), J2.37 (Pin_37), J7.5 (Shield), J8.5 (Shield), J9.5 (Shield), C10.2, C2.1, C25.1, C36.2, C37.2, C8.1, D1.2 (A), D17.1 (K), D19.2 (A), D2.2 (A), D20.2 (A), D21.2 (A), D22.2 (A), D23.2 (A), D24.2 (A), D48.2 (A2), D49.1 (K), D50.1 (K), D52.1 (A), D53.1 (A), D54.1 (A), D55.1 (A), J3.14 (GND), J3.20 (GND), J3.25 (GND), J3.30 (GND), J3.34 (GND), J3.39 (GND), J3.6 (GND), J3.9 (GND), J4.10 (Pin_10), J4.16 (Pin_16), J4.25 (Pin_25), J4.26 (Pin_26), J4.38 (Pin_38), J4.4 (Pin_4), J4.40 (Pin_40), J5.1 (Pin_1), J6.1 (Pin_1), R64.2, R65.2, R80.1, TP5.1, U12.2 (GND), U3.12 (GND), U3.2 (A1), U3.3 (A2); no longer J2.11 (Pin_11), J2.17 (Pin_17), J2.23 (Pin_23), R5.2
- net GPIO0: no longer R18.1
- net GPIO0_OUT: no longer J2.14 (Pin_14), R18.2
- net GPIO1_OUT: now also J2.11 (Pin_11); no longer J2.13 (Pin_13)
- net GPIO2: no longer R23.1
- net GPIO2_OUT: now also J2.14 (Pin_14); no longer J2.20 (Pin_20), R23.2
- net GPIO3_OUT: now also J2.13 (Pin_13); no longer J2.19 (Pin_19)
- net GPIO4: no longer R19.1
- net GPIO4_OUT: no longer J2.26 (Pin_26), R19.2
- net GPIO5: no longer R22.1
- net GPIO5_OUT: no longer J2.25 (Pin_25), R22.2
- net GPIO6_OUT: no longer J2.32 (Pin_32)
- net GPIO7_OUT: now also J2.17 (Pin_17); no longer J2.31 (Pin_31)
- net GPIO_EXT: now also D55.3 (COM), J3.11 (GPIO17/SPI1_~{CE1})
- net RELAY1: now also U3.4 (P00); no longer U2.13 (P10)
- net RELAY2: now also U3.5 (P01); no longer U2.14 (P11)
- net RELAY3: now also U3.6 (P02); no longer U2.15 (P12)
- net RELAY4: now also U3.7 (P03); no longer U2.16 (P13)
- net RPI_D+: now also R22.1, TP11.1
- net RPI_D-: now also R23.1, TP12.1
- net RXD_OUT: now also D2.1 (K), J4.32 (Pin_32); no longer J2.37 (Pin_37)
- net TXD_OUT: now also D1.1 (K), J4.31 (Pin_31); no longer J2.38 (Pin_38)
- net USB_D+: now also TP4.1, U12.3 (I/O2); no longer J1.A6 (D+), J1.B6 (D+)
- net USB_D-: now also TP3.1, U12.1 (I/O1); no longer J1.A7 (D-), J1.B7 (D-)
- net O3D-: now reaches J9.2 (D-), U6.4 (I/O2)
- net O3D+: now reaches J9.3 (D+), U6.6 (I/O1)
- net RELAY4/COM2: now reaches R4.2
- net RELAY4/COM2: no longer R5.1
- net at F1.1, J1.A4 (VBUS), J1.A9 (VBUS)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: now also D48.1 (A1)
- net RELAY2/COM2: now reaches R14.2
- net RELAY3/COM2: now reaches R15.2
- net O2D-: now reaches J8.2 (D-), U5.4 (I/O2)
- net O2D+: now reaches J8.3 (D+), U5.6 (I/O1)
- net RPi_GPIO14: now reaches A1.8 (GP14/TXD), R20.2
- net RPi_GPIO14: now also J3.8 (GPIO14/UART_TXD)
- net at R24.1: now also D24.1 (K), J5.6 (Pin_6)
- net RELAY1/NO2: now reaches D5.2 (A)
- net RELAY1/NO2: no longer D6.1 (K)
- net RELAY2/NO2: now reaches D6.2 (A)
- net O1D-: now reaches J7.2 (D-), U4.4 (I/O2)
- net O1D+: now reaches J7.3 (D+), U4.6 (I/O1)
- net RPi_GPIO15: now reaches A1.10 (GP15/RXD), R21.2
- net RPi_GPIO15: now also J3.10 (GPIO15/UART_RXD)
- net RPi_GPIO18: now reaches A1.12 (GP18)
- net RPi_GPIO18: now also J3.12 (GPIO18/SPI1_~{CE0}/PCM_CLK/PWM0)
- net RPi_GPIO27: now reaches A1.13 (GP27)
- net RPi_GPIO27: now also J3.13 (GPIO27/SDIO_DAT3)
- net RPi_GPIO22: now reaches A1.15 (GP22)
- net RPi_GPIO22: now also J3.15 (GPIO22/SDIO_CLK)
- net RPi_GPIO23: now reaches A1.16 (GP23)
- net RPi_GPIO23: now also J3.16 (GPIO23/SDIO_CMD)
- net RPi_GPIO24: now reaches A1.18 (GP24)
- net RPi_GPIO24: now also J3.18 (GPIO24/SDIO_DAT0)
- net RPi_GPIO10: now reaches A1.19 (GP10/MOSI)
- net RPi_GPIO10: now also J3.19 (MOSI_SPI0/GPIO10)
- net RPi_GPIO9: now reaches A1.21 (GP9/MISO)
- net RPi_GPIO9: now also J3.21 (MISO_SPI0/GPIO09)
- net RPi_GPIO25: now reaches A1.22 (GP25)
- net RPi_GPIO25: now also J3.22 (GPIO25/SDIO_DAT1)
- net RPi_GPIO11: now reaches A1.23 (GP11/SCLK)
- net RPi_GPIO11: now also J3.23 (SCLK_SPI0/GPIO11)
- net RPi_GPIO8: now reaches A1.24 (GP8/CS0)
- net RPi_GPIO8: now also J3.24 (~{CE0}_SPI0/GPIO08)
- net RPi_GPIO7: now reaches A1.26 (GP7/CS1)
- net RPi_GPIO7: now also J3.26 (~{CE1}_SPI0/GPIO07)
- net RPi_GPIO0: now reaches A1.27 (GP0)
- net RPi_GPIO0: now also J3.27 (ID_SD_I2C0/GPIO00)
- net RPi_GPIO1: now reaches A1.28 (GP1)
- net RPi_GPIO1: now also J3.28 (ID_SC_I2C0/GPIO01)
- net RPi_GPIO5: now reaches A1.29 (GP5)
- net RPi_GPIO5: now also R19.2, J3.29 (GPCLK1/GPIO05), U3.1 (~{INT})
- net RPi_GPIO6: now reaches A1.31 (GP6)
- net RPi_GPIO6: now also D22.1 (K), J3.31 (GPCLK2/GPIO06), J5.5 (Pin_5)
- net RPi_GPIO12: now reaches A1.32 (GP12/PWM0)
- net RPi_GPIO12: now also J3.32 (GPIO12/PWM0)
- net RPi_GPIO13: now reaches A1.33 (GP13/PWM1)
- net RPi_GPIO13: now also J3.33 (GPIO13/PWM1)
- net RPi_GPIO19: now reaches A1.35 (GP19)
- net RPi_GPIO19: now also J3.35 (GPIO19/SPI1_MISO/PCM_FS)
- net RPi_GPIO16: now reaches A1.36 (GP16)
- net RPi_GPIO16: now also J3.36 (GPIO16/SPI1_~{CE2})
- net RPi_GPIO26: now reaches A1.37 (GP26)
- net RPi_GPIO26: now also J3.37 (GPIO26/SDIO_DAT2)
- net RPi_GPIO20: now reaches A1.38 (GP20)
- net RPi_GPIO20: now also J3.38 (GPIO20/SPI1_MOSI/PCM_DIN/PWM1)
- net RPi_GPIO21: now reaches A1.40 (GP21)
- net RPi_GPIO21: now also J3.40 (GPIO21/SPI1_SCLK/PCM_DOUT)
- net at C1.2, J1.S1 (SHIELD), R1.1: now also R80.2
- net RELAY4/NO2: now reaches D4.2 (A)
- net COM3 renamed GPIO9_OUT
- net COM4 renamed GPIO15_OUT
- net NC3 renamed GPIO10_OUT
- net NC4: no longer names the net of J2.30 (Pin_30)
- net NO3 renamed GPIO8_OUT
- net NO4 renamed GPIO14_OUT
- net SCL renamed RPi_GPIO3
- net RPi_GPIO3: now also U2.22 (SCL), D20.1 (K), D23.1 (K), D53.3 (COM), J3.5 (SCL_I2C1/GPIO03), J4.28 (Pin_28), J5.4 (Pin_4), J6.4 (Pin_4), TP7.1, U3.22 (SCL); no longer J2.35 (Pin_35), U2.23 (SDA)
- net SDA renamed RPi_GPIO2
- net RPi_GPIO2: now also U2.23 (SDA), D19.1 (K), D21.1 (K), D52.3 (COM), J3.3 (SDA_I2C1/GPIO02), J4.27 (Pin_27), J5.3 (Pin_3), J6.3 (Pin_3), TP6.1, U3.23 (SDA); no longer J2.36 (Pin_36), U2.22 (SCL)
- net USB1_EN renamed GPIO12
- net USB2_EN renamed GPIO13
- net USB3_EN renamed GPIO14
- net USB4_EN renamed GPIO15
- net ~{INT} renamed RPi_GPIO4
- net RPi_GPIO4: now also R18.2, D54.3 (COM), J3.7 (GPCLK0/GPIO04)
- new net: J1.A6 (D+), J1.B6 (D+), U12.4 (I/O2)
- new net: J1.A7 (D-), J1.B7 (D-), U12.6 (I/O1)
- new net: F3.1, J4.37 (Pin_37)
- new net: D15.1 (K), R64.1
- new net: F6.2, J5.2 (Pin_2)
- new net: D49.2 (A), R77.1
- new net: D50.2 (A), R78.1
- new net: F5.2, J6.2 (Pin_2)
- new net: F4.1, J4.39 (Pin_39)
- new net: D16.1 (K), R65.1
- new net: D16.2 (A), U3.11 (P07)
- new net: F8.1, J3.1 (3V3), J3.17 (3V3)
- new net: D15.2 (A), U3.10 (P06)
- new net: F2.1, J3.2 (5V), J3.4 (5V)
- new net ALERT0: U3.8 (P04)
- new net ALERT1: U3.9 (P05)
- new net GPIO10: U2.15 (P12)
- new net GPIO11: U2.16 (P13)
- new net GPIO11_OUT: J2.23 (Pin_23)
- new net GPIO12_OUT: J2.26 (Pin_26)
- new net GPIO13_OUT: J2.25 (Pin_25)
- new net GPIO8: U2.13 (P10)
- new net GPIO9: U2.14 (P11)
- new net RELAY1/COM2: R5.2
- new net RELAY3/NO2: D17.2 (A)
- new net R_COM1: J4.3 (Pin_3)
- new net R_COM2: J4.9 (Pin_9)
- new net R_COM3: J4.15 (Pin_15)
- new net R_COM4: J4.21 (Pin_21)
- new net R_NC1: J4.1 (Pin_1)
- new net R_NC2: J4.7 (Pin_7)
- new net R_NC3: J4.13 (Pin_13)
- new net R_NC4: J4.19 (Pin_19)
- new net R_NO1: J4.5 (Pin_5)
- new net R_NO2: J4.11 (Pin_11)
- new net R_NO3: J4.17 (Pin_17)
- new net R_NO4: J4.23 (Pin_23)
- new net USB_EN1: U3.17 (P14)
- new net USB_EN2: U3.18 (P15)
- new net USB_EN3: U3.19 (P16)
- new net USB_EN4: U3.20 (P17)
- new net USB_FLT1: U3.13 (P10)
- new net USB_FLT2: U3.14 (P11)
- new net USB_FLT3: U3.15 (P12)
- new net USB_FLT4: U3.16 (P13)
- no-connect marks 0 -> 28
Other:
- added sheet ADC0 (pinbot_adc.kicad_sch)
- added sheet ADC1 (pinbot_adc.kicad_sch)
- added sheet Protection (pinbot_protection.kicad_sch)
- added sheet RELAY1 (pinbot_relay.kicad_sch)
- added sheet RELAY2 (pinbot_relay.kicad_sch)
- added sheet RELAY3 (pinbot_relay.kicad_sch)
- added sheet RELAY4 (pinbot_relay.kicad_sch)
- added sheet USBHUB (pinbot_hub.kicad_sch)
- note added: "0x0100001"
- note added: "0x1001000"
- note added: "0x1001001"
- note added: "16ch GPIO 0-24V"
- note added: "4 relays"
- note added: "Adapter board connectors"
- note added: "RPi HAT connector"
- note added: "USB hub & connectors"
- note removed: "1001000"
- note removed: "1001001"
- note removed: "4 Relays"
- note removed: "8ch GPIO 0-24V"
- note removed: "Adapter board connector"
- note removed: "USB-hub with power control"
- title: (none) -> ${PROJECTNAME}
- moved on the sheet: A1, C12, C13, C14, C4, C7, C9, F1, J1, J7, J8, J9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
